Commit message: more computationally-friendly collision geometry
Use simple primitives to replace the fancy mesh
for most parts, except the claw.

Say you want to retain mesh `xyz.stl` and `abc.stl`, you can simply
call `python ./gripper_model.py xyz abc`
(or better modify config.json accordingly)

still missing the contact pad, which shall be relevant for simulation

File: gripper_description/urdf/robot_augmented.urdf (robot description, URDF)
Before this commit: robot parallel_link_gripper, 8 links, 7 joints
Links:
- link body: geometry collision box size=0.008 0.056 0.04; collision box size=0.03 0.003 0.02
- link rod_inner_lhs: geometry collision box size=0.01 0.035 0.005; collision box size=0.012 0.028 0.005
- link rod_inner_rhs: geometry collision box size=0.01 0.035 0.005; collision box size=0.012 0.028 0.005
- link rod_outer: geometry collision box size=0.01 0.038 0.005; visual mesh filename=package://gripper_description/mesh/rod_outer.stl
- link rod_outer_2: geometry collision box size=0.01 0.038 0.005; visual mesh filename=package://gripper_description/mesh/rod_outer.stl

Commit message: enforce naming convention to the links
so that other stuff can be automated more easily
(e.g. gazebo/sdf elements)

File: gripper_description/urdf/robot_augmented.urdf (robot description, URDF)
Before this commit: robot parallel_link_gripper, 8 links, 7 joints
Links:
- removed link jaw
- removed link jaw_2
- removed link rod_inner_lhs
- removed link rod_inner_rhs
- removed link rod_outer
- removed link rod_outer_2
- added link lhs_claw, mass 0.0692262; collision mesh filename=package://gripper_description/mesh/jaw_plate.stl; visual mesh filename=package://gripper_description/mesh/jaw_plate.stl
- added link lhs_inner_beam, mass 0.008336; collision box size=0.01 0.035 0.005; collision box size=0.012 0.028 0.005
- added link lhs_outer_beam, mass 0.00147516; collision box size=0.01 0.038 0.005; visual mesh filename=package://gripper_description/mesh/rod_outer.stl
- added link rhs_claw, mass 0.0692262; collision mesh filename=package://gripper_description/mesh/jaw_plate.stl; visual mesh filename=package://gripper_description/mesh/jaw_plate.stl
- added link rhs_inner_beam, mass 0.00680759; collision box size=0.01 0.035 0.005; collision box size=0.012 0.028 0.005
- added link rhs_outer_beam, mass 0.00147516; collision box size=0.01 0.038 0.005; visual mesh filename=package://gripper_description/mesh/rod_outer.stl
Joints:
- joint lhs_j1: child rod_inner_lhs -> lhs_inner_beam
- joint lhs_j2: child rod_outer -> lhs_outer_beam
- joint lhs_j3: child jaw -> lhs_claw; parent rod_inner_lhs -> lhs_inner_beam
- joint rhs_j1: child rod_inner_rhs -> rhs_inner_beam
- joint rhs_j2: child rod_outer_2 -> rhs_outer_beam
- joint rhs_j3: child jaw_2 -> rhs_claw; parent rod_inner_rhs -> rhs_inner_beam

Commit message: lengthened the beams from 3 cm to 3.5 cm, also added form closure

File: gripper_description/urdf/robot_augmented.urdf (robot description, URDF)
Before this commit: robot parallel_link_gripper, 8 links, 7 joints
Links:
- link body: geometry collision box size=0.008 0.048 0.04; collision box size=0.03 0.003 0.02
- link lhs_claw: mass 0.0692262 -> 0.0706194
- link lhs_inner_beam: mass 0.008336 -> 0.00897747; geometry collision box size=0.01 0.039 0.005; collision box size=0.012 0.036 0.005
- link lhs_outer_beam: mass 0.00147516 -> 0.00168556; geometry collision box size=0.01 0.043 0.005; visual mesh filename=package://gripper_description/mesh/rod_outer.stl
- link rhs_claw: mass 0.0692262 -> 0.0706194
- link rhs_inner_beam: mass 0.00680759 -> 0.00744734; geometry collision box size=0.01 0.039 0.005; collision box size=0.012 0.036 0.005
- link rhs_outer_beam: mass 0.00147516 -> 0.00168556; geometry collision box size=0.01 0.043 0.005; visual mesh filename=package://gripper_description/mesh/rod_outer.stl
Joints:
- joint lhs_j1: origin xyz=0.03725 0.015 0.017 rpy=-1.9792e-14 -3.38332e-16 -3.14159 -> xyz=0.03725 0.015 0.017 rpy=-1.9792e-14 -6.27246e-15 -3.14159
- joint lhs_j2: origin xyz=0.01725 0.04 -1.25421e-15 rpy=-3.14159 -6.16349e-16 5.9816e-13 -> xyz=0.01725 0.04 -1.249e-15 rpy=-3.14159 4.40184e-15 7.06094e-13
- joint lhs_j3: origin xyz=0 -0.03 -0.017 rpy=-1.3685e-16 3.07629e-16 3.14159 -> xyz=-1.38778e-17 -0.035 -0.017 rpy=1.32156e-16 -3.87474e-17 3.14159
- joint rhs_j1: origin xyz=0.03725 -0.015 -1.6679e-19 rpy=-3.14417e-16 2.28667e-16 -1.5708 -> xyz=0.03725 -0.015 8.67246e-31 rpy=-6.24854e-15 1.67434e-16 -1.5708
- joint rhs_j2: origin xyz=0.01725 -0.04 0 rpy=-3.14159 -4.12648e-15 5.65242e-14 -> xyz=0.01725 -0.04 -3.46945e-18 rpy=-3.14159 6.24854e-15 -5.22162e-14
- joint rhs_j3: origin xyz=0.03 1.38778e-17 -3.46945e-18 rpy=-3.14159 -8.55478e-24 1.5708 -> xyz=0.035 6.93889e-18 -3.46945e-18 rpy=-3.14159 -0 1.5708
