Commit message: further reduced the 0-DoF gripper into just 1 link
* total mass indeed equivalent to the unfrozen version
* passed visual inspection with rviz

File: gripper_description/urdf/gripper_0dof.reusable.xacro (robot description, xacro)
@@ -1,13 +1,12 @@
 <robot name="parallel_link_gripper" xmlns:xacro="http://www.ros.org/wiki/xacro">
   <xacro:macro name="mk_parallel_gripper_with_0dof" params="ns">
-    <link name="${ns}/base_link" />
-    <joint name="${ns}/base_link_to_base" type="fixed">
-      <parent link="${ns}/base_link" />
-      <child link="${ns}/body" />
-      <origin rpy="0 0 0" xyz="0 0 0" />
-    </joint>
-    <link name="${ns}/body">
-      <visual>
-        <origin xyz="0.002 0 -0.017" rpy="0 0 0" />
+    <link name="${ns}/base_link">
+      <inertial>
+        <mass value="0.31845672999999997" />
+        <origin xyz="0.04539854906879699 0.00439535282382325 0.00023774165341415557" rpy="0.0 -0.0 0.0" />
+        <inertia ixx="0.0006409486799300743" iyy="0.0005001150057078902" izz="0.0010633935422334798" ixy="7.585469594750223e-06" ixz="-6.942599742535248e-06" iyz="6.949343630899062e-06" />
+      </inertial>
+      <visual>
+        <origin xyz="0.002 0.0 -0.017" rpy="0.0 -0.0 0.0" />
         <geometry>
           <mesh filename="package://gripper_description/mesh/gripper_mount__list_gggmxkb4ygsnke_default.stl" />
@@ -17,18 +16,6 @@
         </material>
       </visual>
-      <collision>
-        <origin xyz="0.0205 0 0" rpy="0 0 0" />
-        <geometry>
-          <box size="0.041 0.066 0.04" />
-        </geometry>
-      </collision>
-      <collision>
-        <origin xyz="0.045 0 0" rpy="0 0 0" />
-        <geometry>
-          <box size="0.008 0.048 0.04" />
-        </geometry>
-      </collision>
-      <visual>
-        <origin xyz="0.002 0 -0.017" rpy="0 0 0" />
+      <visual>
+        <origin xyz="0.002 0.0 -0.017" rpy="0.0 -0.0 0.0" />
         <geometry>
           <mesh filename="package://gripper_description/mesh/gripper_x430_shell_rhs__list_gggmxkb4ygsnke_default.stl" />
@@ -39,5 +26,5 @@
       </visual>
       <visual>
-        <origin xyz="0.002 0 -0.017" rpy="0 0 0" />
+        <origin xyz="0.002 0.0 -0.017" rpy="0.0 -0.0 0.0" />
         <geometry>
           <mesh filename="package://gripper_description/mesh/gripper_bracket_rhs__list_gggmxkb4ygsnke_default.stl" />
@@ -47,18 +34,6 @@
         </material>
       </visual>
-      <collision>
-        <origin xyz="0.0215 -0.034 0" rpy="0 0 0" />
-        <geometry>
-          <box size="0.03 0.003 0.02" />
-        </geometry>
-      </collision>
-      <collision>
-        <origin xyz="0.0173 -0.04 0" rpy="0 0 0" />
-        <geometry>
-          <cylinder length="0.02" radius="0.005" />
-        </geometry>
-      </collision>
-      <visual>
-        <origin xyz="0.03725 0.015 0.019" rpy="0 0 -1.5708" />
+      <visual>
+        <origin xyz="0.03725 0.015 0.019" rpy="0.0 -0.0 -1.5708" />
         <geometry>
           <mesh filename="package://gripper_description/mesh/dynamixel_casing__list_ndk53xfpevccij_default.stl" />
@@ -69,5 +44,5 @@
       </visual>
       <visual>
-        <origin xyz="0.002 0.0615 -0.017" rpy="0 0 0" />
+        <origin xyz="0.002 0.0615 -0.017" rpy="0.0 -0.0 0.0" />
         <geometry>
           <mesh filename="package://gripper_description/mesh/gripper_bracket_pad__list_gggmxkb4ygsnke_default.stl" />
@@ -77,12 +52,6 @@
         </material>
       </visual>
-      <collision>
-        <origin xyz="0.0215 0.0307 0" rpy="0 0 0" />
-        <geometry>
-          <box size="0.03 0.003 0.02" />
-        </geometry>
-      </collision>
-      <visual>
-        <origin xyz="0.002 0 0.017" rpy="-3.14159 0 0" />
+      <visual>
+        <origin xyz="0.002 0.0 0.017" rpy="-3.14159 -0.0 0.0" />
         <geometry>
           <mesh filename="package://gripper_description/mesh/gripper_bracket_rhs__list_gggmxkb4ygsnke_default.stl" />
@@ -93,5 +62,17 @@
       </visual>
       <collision>
-        <origin xyz="0.0215 0.034 0" rpy="-3.14159 0 0" />
+        <origin xyz="0.0205 0.0 0.0" rpy="0.0 -0.0 0.0" />
+        <geometry>
+          <box size="0.041 0.066 0.04" />
+        </geometry>
+      </collision>
+      <collision>
+        <origin xyz="0.045 0.0 0.0" rpy="0.0 -0.0 0.0" />
+        <geometry>
+          <box size="0.008 0.048 0.04" />
+        </geometry>
+      </collision>
+      <collision>
+        <origin xyz="0.0215 -0.034 0.0" rpy="0.0 -0.0 0.0" />
         <geometry>
           <box size="0.03 0.003 0.02" />
@@ -99,18 +80,29 @@
       </collision>
       <collision>
-        <origin xyz="0.0173 0.04 0" rpy="-3.14159 0 0" />
+        <origin xyz="0.0173 -0.04 0.0" rpy="0.0 -0.0 0.0" />
         <geometry>
           <cylinder length="0.02" radius="0.005" />
         </geometry>
       </collision>
-      <inertial>
-        <origin xyz="0.0224723 0.00874655 0.000222665" rpy="0 0 0" />
-        <mass value="0.157422" />
-        <inertia ixx="6.18655e-05" ixy="-4.90692e-06" ixz="1.13998e-08" iyy="5.05121e-05" iyz="-2.19198e-07" izz="7.60343e-05" />
-      </inertial>
-    </link>
-    <link name="${ns}/lhs_inner_beam">
-      <visual>
-        <origin xyz="0 0.015 -0.017" rpy="0 0 3.14159" />
+      <collision>
+        <origin xyz="0.0215 0.0307 0.0" rpy="0.0 -0.0 0.0" />
+        <geometry>
+          <box size="0.03 0.003 0.02" />
+        </geometry>
+      </collision>
+      <collision>
+        <origin xyz="0.0215 0.034 0.0" rpy="-3.14159 -0.0 0.0" />
+        <geometry>
+          <box size="0.03 0.003 0.02" />
+        </geometry>
+      </collision>
+      <collision>
+        <origin xyz="0.0173 0.04 0.0" rpy="-3.14159 -0.0 0.0" />
+        <geometry>
+          <cylinder length="0.02" radius="0.005" />
+        </geometry>
+      </collision>
+      <visual>
+        <origin xyz="0.026643426427809192 0.004393370136669067 0.0" rpy="-0.0 -0.0 -0.7853981633974481" />
         <geometry>
           <mesh filename="package://gripper_description/mesh/rod_inner_lhs_top.stl" />
@@ -120,18 +112,6 @@
         </material>
       </visual>
-      <collision>
-        <origin xyz="0 0 0.0045" rpy="0 0 3.14159" />
-        <geometry>
-          <cylinder length="0.005" radius="0.013" />
-        </geometry>
-      </collision>
-      <collision>
-        <origin xyz="0 -0.0195 0.0045" rpy="0 0 3.14159" />
-        <geometry>
-          <box size="0.01 0.039 0.005" />
-        </geometry>
-      </collision>
-      <visual>
-        <origin xyz="0 0.015 -0.024" rpy="0 0 0" />
+      <visual>
+        <origin xyz="0.026643426427809192 0.004393370136669067 -0.006999999999999999" rpy="0.0 -0.0 2.3561971437821385" />
         <geometry>
           <mesh filename="package://gripper_description/mesh/rod_inner_bottom.stl" />
@@ -141,18 +121,6 @@
         </material>
       </visual>
-      <collision>
-        <origin xyz="0 -0.02 -0.039" rpy="0 0 0" />
-        <geometry>
-          <box size="0.012 0.036 0.005" />
-        </geometry>
-      </collision>
-      <collision>
-        <origin xyz="0 0 -0.039" rpy="0 0 0" />
-        <geometry>
-          <cylinder length="0.005" radius="0.011" />
-        </geometry>
-      </collision>
-      <visual>
-        <origin xyz="0 0 0.002" rpy="0 0 0" />
+      <visual>
+        <origin xyz="0.03725 0.015 0.019000000000000003" rpy="0.0 -0.0 2.3561971437821385" />
         <geometry>
           <mesh filename="package://gripper_description/mesh/dynamixel_horn__list_ndk53xfpevccij_default.stl" />
@@ -162,48 +130,48 @@
         </material>
       </visual>
-      <inertial>
-        <origin xyz="-0.000694637 -0.00752629 -0.013178" rpy="0 0 0" />
-        <mass value="0.00897747" />
-        <inertia ixx="5.34685e-06" ixy="4.25659e-08" ixz="1.10241e-07" iyy="4.1093e-06" iyz="-5.49535e-07" izz="1.77758e-06" />
-      </inertial>
-    </link>
-    <link name="${ns}/lhs_claw">
-      <visual>
-        <origin xyz="0 -0.006 0" rpy="0 0 0" />
-        <geometry>
-          <mesh filename="package://gripper_description/mesh/jaw_plate.stl" />
-        </geometry>
-        <material name="jaw_plate_material">
-          <color rgba="0.980392 0.796078 0.262745 1.0" />
-        </material>
-      </visual>
-      <collision>
-        <origin xyz="0 -0.006 0" rpy="0 0 0" />
-        <geometry>
-          <mesh filename="package://gripper_description/mesh/jaw_plate.stl" />
-        </geometry>
-        <material name="jaw_plate_material">
-          <color rgba="0.980392 0.796078 0.262745 1.0" />
-        </material>
-      </collision>
-      <inertial>
-        <origin xyz="0.00954335 0.0109092 -3.55182e-09" rpy="0 0 0" />
-        <mass value="0.0706194" />
-        <inertia ixx="1.06828e-05" ixy="6.2682e-06" ixz="0" iyy="3.9212e-05" iyz="1.29448e-11" izz="3.75191e-05" />
-      </inertial>
-    </link>
-    <joint name="${ns}/lhs_j3" type="fixed">
-      <origin xyz="0.0 -0.035 -0.017" rpy="0.0 -0.0 -2.3561971437821385" />
-      <parent link="${ns}/lhs_inner_beam" />
-      <child link="${ns}/lhs_claw" />
-    </joint>
-    <joint name="${ns}/lhs_j1" type="fixed">
-      <origin xyz="0.03725 0.015 0.017" rpy="0.0 -0.0 2.3561971437821385" />
-      <parent link="${ns}/base_link" />
-      <child link="${ns}/lhs_inner_beam" />
-    </joint>
-    <link name="${ns}/lhs_outer_beam">
-      <visual>
-        <origin xyz="0.02 0.025 0.0025" rpy="-3.14159 0 0" />
+      <visual>
+        <origin xyz="0.06199867166844522 0.03374880301443885 0.0" rpy="-0.0 -0.0 -2.1438260709158268e-18" />
+        <geometry>
+          <mesh filename="package://gripper_description/mesh/jaw_plate.stl" />
+        </geometry>
+        <material name="jaw_plate_material">
+          <color rgba="0.980392 0.796078 0.262745 1.0" />
+        </material>
+      </visual>
+      <collision>
+        <origin xyz="0.03725 0.015 0.021500000000000002" rpy="-0.0 -0.0 -0.7853981633974481" />
+        <geometry>
+          <cylinder length="0.005" radius="0.013" />
+        </geometry>
+      </collision>
+      <collision>
+        <origin xyz="0.05103854564384805 0.028788618822330213 0.021500000000000002" rpy="-0.0 -0.0 -0.7853981633974481" />
+        <geometry>
+          <box size="0.01 0.039 0.005" />
+        </geometry>
+      </collision>
+      <collision>
+        <origin xyz="0.051392098096254404 0.02914217315110791 -0.022" rpy="0.0 -0.0 2.3561971437821385" />
+        <geometry>
+          <box size="0.012 0.036 0.005" />
+        </geometry>
+      </collision>
+      <collision>
+        <origin xyz="0.03725 0.015 -0.022" rpy="0.0 -0.0 2.3561971437821385" />
+        <geometry>
+          <cylinder length="0.005" radius="0.011" />
+        </geometry>
+      </collision>
+      <collision>
+        <origin xyz="0.06199867166844522 0.03374880301443885 0.0" rpy="-0.0 -0.0 -2.1438260709158268e-18" />
+        <geometry>
+          <mesh filename="package://gripper_description/mesh/jaw_plate.stl" />
+        </geometry>
+        <material name="jaw_plate_material">
+          <color rgba="0.980392 0.796078 0.262745 1.0" />
+        </material>
+      </collision>
+      <visual>
+        <origin xyz="0.013714466094067266 0.008180201480691873 -0.002500084436701384" rpy="4.529961130895335e-06 1.8763713373682258e-06 -0.7853981633956878" />
         <geometry>
           <mesh filename="package://gripper_description/mesh/rod_outer.stl" />
@@ -214,23 +182,11 @@
       </visual>
       <collision>
-        <origin xyz="0 -0.0175 0" rpy="-3.14159 0 0" />
+        <origin xyz="0.02962436867076458 0.05237436867072102 3.283649840686403e-08" rpy="4.529961130895335e-06 1.8763713373682258e-06 -0.7853981633956878" />
         <geometry>
           <box size="0.01 0.043 0.005" />
         </geometry>
       </collision>
-      <inertial>
-        <origin xyz="0 -0.0175 0" rpy="0 0 0" />
-        <mass value="0.00168556" />
-        <inertia ixx="2.35764e-07" ixy="0" ixz="0" iyy="1.24039e-08" iyz="0" izz="2.41145e-07" />
-      </inertial>
-    </link>
-    <joint name="${ns}/lhs_j2" type="fixed">
-      <origin xyz="0.01725 0.04 0.0" rpy="-3.1415907772184557 1.8763713373682256e-06 -0.7853981633956878" />
-      <parent link="${ns}/base_link" />
-      <child link="${ns}/lhs_outer_beam" />
-    </joint>
-    <link name="${ns}/rhs_inner_beam">
-      <visual>
-        <origin xyz="-0.015 0 0" rpy="0 0 1.5708" />
+      <visual>
+        <origin xyz="0.0266434372424969 -0.004393359322049782 0.0" rpy="0.0 0.0 0.7853981633974483" />
         <geometry>
           <mesh filename="package://gripper_description/mesh/rod_inner_rhs_top.stl" />
@@ -240,18 +196,6 @@
         </material>
       </visual>
-      <collision>
-        <origin xyz="0 0 0.0215" rpy="0 0 1.5708" />
-        <geometry>
-          <cylinder length="0.005" radius="0.013" />
-        </geometry>
-      </collision>
-      <collision>
-        <origin xyz="0.0195 0 0.0215" rpy="0 0 1.5708" />
-        <geometry>
-          <box size="0.01 0.039 0.005" />
-        </geometry>
-      </collision>
-      <visual>
-        <origin xyz="-0.015 0 -0.007" rpy="0 0 1.5708" />
+      <visual>
+        <origin xyz="0.0266434372424969 -0.004393359322049782 -0.007" rpy="0.0 0.0 0.7853981633974483" />
         <geometry>
           <mesh filename="package://gripper_description/mesh/rod_inner_bottom.stl" />
@@ -261,6 +205,27 @@
         </material>
       </visual>
-      <collision>
-        <origin xyz="0.02 0 -0.022" rpy="0 0 1.5708" />
+      <visual>
+        <origin xyz="0.06199864643418446 -0.03374882824856107 1.1258228025210527e-08" rpy="-3.1415907772184557 1.8763713373682256e-06 1.7603916580989416e-12" />
+        <geometry>
+          <mesh filename="package://gripper_description/mesh/jaw_plate.stl" />
+        </geometry>
+        <material name="jaw_plate_material">
+          <color rgba="0.980392 0.796078 0.262745 1.0" />
+        </material>
+      </visual>
+      <collision>
+        <origin xyz="0.03725 -0.015 0.0215" rpy="0.0 0.0 0.7853981633974483" />
+        <geometry>
+          <cylinder length="0.005" radius="0.013" />
+        </geometry>
+      </collision>
+      <collision>
+        <origin xyz="0.05103853158475403 -0.028788632881335284 0.0215" rpy="0.0 0.0 0.7853981633974483" />
+        <geometry>
+          <box size="0.01 0.039 0.005" />
+        </geometry>
+      </collision>
+      <collision>
+        <origin xyz="0.051392083676670794 -0.02914218757060029 -0.022" rpy="0.0 0.0 0.7853981633974483" />
         <geometry>
           <box size="0.012 0.036 0.005" />
@@ -268,53 +233,20 @@
       </collision>
       <collision>
-        <origin xyz="0 0 -0.022" rpy="0 0 1.5708" />
+        <origin xyz="0.03725 -0.015 -0.022" rpy="0.0 0.0 0.7853981633974483" />
         <geometry>
           <cylinder length="0.005" radius="0.011" />
         </geometry>
       </collision>
-      <inertial>
-        <origin xyz="0.00901442 0.000756382 0.000852503" rpy="0 0 0" />
-        <mass value="0.00744734" />
-        <inertia ixx="3.68765e-06" ixy="4.3779e-08" ixz="3.57846e-07" iyy="4.8283e-06" iyz="-1.16308e-07" izz="1.61067e-06" />
-      </inertial>
-    </link>
-    <link name="${ns}/rhs_claw">
-      <visual>
-        <origin xyz="0 -0.006 0" rpy="0 0 0" />
-        <geometry>
-          <mesh filename="package://gripper_description/mesh/jaw_plate.stl" />
-        </geometry>
-        <material name="jaw_plate_material">
-          <color rgba="0.980392 0.796078 0.262745 1.0" />
-        </material>
-      </visual>
-      <collision>
-        <origin xyz="0 -0.006 0" rpy="0 0 0" />
-        <geometry>
-          <mesh filename="package://gripper_description/mesh/jaw_plate.stl" />
-        </geometry>
-        <material name="jaw_plate_material">
-          <color rgba="0.980392 0.796078 0.262745 1.0" />
-        </material>
-      </collision>
-      <inertial>
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