Commit message: ROS Control stuff & simulation
* added <transmission> to the reusable xacro:macro
* gazebo_ros_control stuff
  * joint state "measurement" publishing (to ROS)
  * physics-based servo actuator model.
    ...
    Parameters to be calibrated/ corrected:
    * joint limits (velocity & torque)
    * joint friction params
    * the PID model of the controller

In general, see the revised launch scripts
for more details.

File: gripper_description/urdf/gripper.reusable.xacro (robot description, xacro)
@@ -364,4 +364,13 @@
       <mimic joint="${ns}/lhs_j1" multiplier="1" offset="0" />
     </joint>
+    <transmission name="${ns}/lhs_j1_transmission">
+      <type>transmission_interface/SimpleTransmission</type>
+      <joint name="${ns}/lhs_j1">
+        <hardwareInterface>hardware_interface/PositionJointInterface</hardwareInterface>
+      </joint>
+      <actuator name="${ns}/lhs_j1_actuator">
+        <mechanicalReduction>1</mechanicalReduction>
+      </actuator>
+    </transmission>
   </xacro:macro>
 </robot>

File: gripper_gazebo/sdf/gripper_fixed.xacro (robot description, xacro)
@@ -10,4 +10,7 @@
   <xacro:gripper_friction_lining ns="$(arg namespace)" prefix="rhs" />
   <gazebo>
+    <plugin name="gazebo_ros_control" filename="libgazebo_ros_control.so">
+      <robotNamespace>$(arg namespace)</robotNamespace>
+    </plugin>
     <self_collide>true</self_collide>
     <!-- https://answers.ros.org/question/393006/urdf-link-not-properly-fixed-to-world/ -->

Commit message: regenerated the URDF with structural zeros whenever reasonable

File: gripper_description/urdf/gripper.reusable.xacro (robot description, xacro)
@@ -5,9 +5,9 @@
       <parent link="${ns}/base_link" />
       <child link="${ns}/body" />
-      <origin rpy="0.0 0 0" xyz="0 0 0" />
+      <origin rpy="0 0 0" xyz="0 0 0" />
     </joint>
     <link name="${ns}/body">
       <visual>
-        <origin xyz="0.002 2.84109e-20 -0.017" rpy="4.43272e-17 9.56494e-30 -6.02851e-29" />
+        <origin xyz="0.002 0 -0.017" rpy="0 0 0" />
         <geometry>
           <mesh filename="package://gripper_description/mesh/gripper_mount__list_gggmxkb4ygsnke_default.stl" />
@@ -18,5 +18,5 @@
       </visual>
       <collision>
-        <origin xyz="0.0205 2.84109e-20 -6.93889e-18" rpy="4.43272e-17 9.56494e-30 -6.02851e-29" />
+        <origin xyz="0.0205 0 0" rpy="0 0 0" />
         <geometry>
           <box size="0.041 0.066 0.04" />
@@ -24,5 +24,5 @@
       </collision>
       <collision>
-        <origin xyz="0.045 2.84109e-20 -6.93889e-18" rpy="4.43272e-17 9.56494e-30 -6.02851e-29" />
+        <origin xyz="0.045 0 0" rpy="0 0 0" />
         <geometry>
           <box size="0.008 0.048 0.04" />
@@ -30,5 +30,5 @@
       </collision>
       <visual>
-        <origin xyz="0.002 1.04368e-17 -0.017" rpy="2.72994e-16 3.14417e-16 -6.18698e-29" />
+        <origin xyz="0.002 0 -0.017" rpy="0 0 0" />
         <geometry>
           <mesh filename="package://gripper_description/mesh/gripper_x430_shell_rhs__list_gggmxkb4ygsnke_default.stl" />
@@ -39,5 +39,5 @@
       </visual>
       <visual>
-        <origin xyz="0.002 1.73756e-17 -0.017" rpy="2.72994e-16 3.14417e-16 -6.18698e-29" />
+        <origin xyz="0.002 0 -0.017" rpy="0 0 0" />
         <geometry>
           <mesh filename="package://gripper_description/mesh/gripper_bracket_rhs__list_gggmxkb4ygsnke_default.stl" />
@@ -48,5 +48,5 @@
       </visual>
       <collision>
-        <origin xyz="0.0215 -0.034 0" rpy="2.72994e-16 3.14417e-16 -6.18698e-29" />
+        <origin xyz="0.0215 -0.034 0" rpy="0 0 0" />
         <geometry>
           <box size="0.03 0.003 0.02" />
@@ -54,5 +54,5 @@
       </collision>
       <collision>
-        <origin xyz="0.0173 -0.04 0" rpy="2.72994e-16 3.14417e-16 -6.18698e-29" />
+        <origin xyz="0.0173 -0.04 0" rpy="0 0 0" />
         <geometry>
           <cylinder length="0.02" radius="0.005" />
@@ -60,5 +60,5 @@
       </collision>
       <visual>
-        <origin xyz="0.03725 0.015 0.019" rpy="-4.91725e-16 1.98363e-14 -1.5708" />
+        <origin xyz="0.03725 0.015 0.019" rpy="0 0 -1.5708" />
         <geometry>
           <mesh filename="package://gripper_description/mesh/dynamixel_casing__list_ndk53xfpevccij_default.stl" />
@@ -69,5 +69,5 @@
       </visual>
       <visual>
-        <origin xyz="0.002 0.0615 -0.017" rpy="2.72994e-16 3.71583e-16 7.45931e-17" />
+        <origin xyz="0.002 0.0615 -0.017" rpy="0 0 0" />
         <geometry>
           <mesh filename="package://gripper_description/mesh/gripper_bracket_pad__list_gggmxkb4ygsnke_default.stl" />
@@ -78,5 +78,5 @@
       </visual>
       <collision>
-        <origin xyz="0.0215 0.0307 3.81639e-17" rpy="2.72994e-16 3.71583e-16 7.45931e-17" />
+        <origin xyz="0.0215 0.0307 0" rpy="0 0 0" />
         <geometry>
           <box size="0.03 0.003 0.02" />
@@ -84,5 +84,5 @@
       </collision>
       <visual>
-        <origin xyz="0.002 -1.8235e-17 0.017" rpy="-3.14159 3.14417e-16 5.37331e-16" />
+        <origin xyz="0.002 0 0.017" rpy="-3.14159 0 0" />
         <geometry>
           <mesh filename="package://gripper_description/mesh/gripper_bracket_rhs__list_gggmxkb4ygsnke_default.stl" />
@@ -93,5 +93,5 @@
       </visual>
       <collision>
-        <origin xyz="0.0215 0.034 -1.25247e-15" rpy="-3.14159 3.14417e-16 5.37331e-16" />
+        <origin xyz="0.0215 0.034 0" rpy="-3.14159 0 0" />
         <geometry>
           <box size="0.03 0.003 0.02" />
@@ -99,5 +99,5 @@
       </collision>
       <collision>
-        <origin xyz="0.0173 0.04 -1.249e-15" rpy="-3.14159 3.14417e-16 5.37331e-16" />
+        <origin xyz="0.0173 0.04 0" rpy="-3.14159 0 0" />
         <geometry>
           <cylinder length="0.02" radius="0.005" />
@@ -112,5 +112,5 @@
     <link name="${ns}/lhs_inner_beam">
       <visual>
-        <origin xyz="6.93889e-18 0.015 -0.017" rpy="1.32156e-16 -3.87474e-17 3.14159" />
+        <origin xyz="0 0.015 -0.017" rpy="0 0 3.14159" />
         <geometry>
           <mesh filename="package://gripper_description/mesh/rod_inner_lhs_top.stl" />
@@ -121,5 +121,5 @@
       </visual>
       <collision>
-        <origin xyz="2.35963e-18 1.73472e-18 0.0045" rpy="1.32156e-16 -3.87474e-17 3.14159" />
+        <origin xyz="0 0 0.0045" rpy="0 0 3.14159" />
         <geometry>
           <cylinder length="0.005" radius="0.013" />
@@ -127,5 +127,5 @@
       </collision>
       <collision>
-        <origin xyz="-4.67641e-18 -0.0195 0.0045" rpy="1.32156e-16 -3.87474e-17 3.14159" />
+        <origin xyz="0 -0.0195 0.0045" rpy="0 0 3.14159" />
         <geometry>
           <box size="0.01 0.039 0.005" />
@@ -133,5 +133,5 @@
       </collision>
       <visual>
-        <origin xyz="1.38778e-17 0.015 -0.024" rpy="-1.46561e-16 3.87474e-17 -4.71845e-16" />
+        <origin xyz="0 0.015 -0.024" rpy="0 0 0" />
         <geometry>
           <mesh filename="package://gripper_description/mesh/rod_inner_bottom.stl" />
@@ -142,5 +142,5 @@
       </visual>
       <collision>
-        <origin xyz="-3.21799e-18 -0.02 -0.039" rpy="-1.46561e-16 3.87474e-17 -4.71845e-16" />
+        <origin xyz="0 -0.02 -0.039" rpy="0 0 0" />
         <geometry>
           <box size="0.012 0.036 0.005" />
@@ -148,5 +148,5 @@
       </collision>
       <collision>
-        <origin xyz="6.2189e-18 -5.20417e-18 -0.039" rpy="1.46561e-16 3.87474e-17 -4.71845e-16" />
+        <origin xyz="0 0 -0.039" rpy="0 0 0" />
         <geometry>
           <cylinder length="0.005" radius="0.011" />
@@ -154,5 +154,5 @@
       </collision>
       <visual>
-        <origin xyz="0 0 0.002" rpy="0 -0 -2.31702e-29" />
+        <origin xyz="0 0 0.002" rpy="0 0 0" />
         <geometry>
           <mesh filename="package://gripper_description/mesh/dynamixel_horn__list_ndk53xfpevccij_default.stl" />
@@ -170,5 +170,5 @@
     <link name="${ns}/lhs_claw">
       <visual>
-        <origin xyz="0 -0.006 -1.97215e-31" rpy="0 -0 2.01638e-30" />
+        <origin xyz="0 -0.006 0" rpy="0 0 0" />
         <geometry>
           <mesh filename="package://gripper_description/mesh/jaw_plate.stl" />
@@ -179,5 +179,5 @@
       </visual>
       <collision>
-        <origin xyz="0 -0.006 -1.97215e-31" rpy="0 -0 2.01638e-30" />
+        <origin xyz="0 -0.006 0" rpy="0 0 0" />
         <geometry>
           <mesh filename="package://gripper_description/mesh/jaw_plate.stl" />
@@ -190,9 +190,9 @@
         <origin xyz="0.00954335 0.0109092 -3.55182e-09" rpy="0 0 0" />
         <mass value="0.0706194" />
-        <inertia ixx="1.06828e-05" ixy="6.2682e-06" ixz="7.52244e-13" iyy="3.9212e-05" iyz="1.29448e-11" izz="3.75191e-05" />
+        <inertia ixx="1.06828e-05" ixy="6.2682e-06" ixz="0" iyy="3.9212e-05" iyz="1.29448e-11" izz="3.75191e-05" />
       </inertial>
     </link>
     <joint name="${ns}/lhs_j3" type="continuous">
-      <origin xyz="-1.38778e-17 -0.035 -0.017" rpy="1.32156e-16 -3.87474e-17 3.14159" />
+      <origin xyz="0 -0.035 -0.017" rpy="0 0 3.14159" />
       <parent link="${ns}/lhs_inner_beam" />
       <child link="${ns}/lhs_claw" />
@@ -203,5 +203,5 @@
     </joint>
     <joint name="${ns}/lhs_j1" type="revolute">
-      <origin xyz="0.03725 0.015 0.017" rpy="-1.9792e-14 -6.27246e-15 -3.14159" />
+      <origin xyz="0.03725 0.015 0.017" rpy="0 0 -3.14159" />
       <parent link="${ns}/base_link" />
       <child link="${ns}/lhs_inner_beam" />
@@ -212,5 +212,5 @@
     <link name="${ns}/lhs_outer_beam">
       <visual>
-        <origin xyz="0.02 0.025 0.0025" rpy="-3.14159 -1.88544e-31 3.5742e-29" />
+        <origin xyz="0.02 0.025 0.0025" rpy="-3.14159 0 0" />
         <geometry>
           <mesh filename="package://gripper_description/mesh/rod_outer.stl" />
@@ -221,5 +221,5 @@
       </visual>
       <collision>
-        <origin xyz="3.46945e-18 -0.0175 0" rpy="-3.14159 -1.88544e-31 3.5742e-29" />
+        <origin xyz="0 -0.0175 0" rpy="-3.14159 0 0" />
         <geometry>
           <box size="0.01 0.043 0.005" />
@@ -227,11 +227,11 @@
       </collision>
       <inertial>
-        <origin xyz="3.46945e-18 -0.0175 0" rpy="0 0 0" />
+        <origin xyz="0 -0.0175 0" rpy="0 0 0" />
         <mass value="0.00168556" />
-        <inertia ixx="2.35764e-07" ixy="8.3159e-36" ixz="9.11279e-38" iyy="1.24039e-08" iyz="-3.0331e-37" izz="2.41145e-07" />
+        <inertia ixx="2.35764e-07" ixy="0" ixz="0" iyy="1.24039e-08" iyz="0" izz="2.41145e-07" />
       </inertial>
     </link>
     <joint name="${ns}/lhs_j2" type="continuous">
-      <origin xyz="0.01725 0.04 -1.249e-15" rpy="-3.14159 4.40184e-15 7.06094e-13" />
+      <origin xyz="0.01725 0.04 0" rpy="-3.14159 0 0" />
       <parent link="${ns}/base_link" />
       <child link="${ns}/lhs_outer_beam" />
@@ -243,5 +243,5 @@
     <link name="${ns}/rhs_inner_beam">
       <visual>
-        <origin xyz="-0.015 6.93889e-18 -3.46945e-18" rpy="0 -0 1.5708" />
+        <origin xyz="-0.015 0 0" rpy="0 0 1.5708" />
         <geometry>
           <mesh filename="package://gripper_description/mesh/rod_inner_rhs_top.stl" />
@@ -252,5 +252,5 @@
       </visual>
       <collision>
-        <origin xyz="0 6.93889e-18 0.0215" rpy="0 -0 1.5708" />
+        <origin xyz="0 0 0.0215" rpy="0 0 1.5708" />
         <geometry>
           <cylinder length="0.005" radius="0.013" />
@@ -258,5 +258,5 @@
       </collision>
       <collision>
-        <origin xyz="0.0195 6.93889e-18 0.0215" rpy="0 -0 1.5708" />
+        <origin xyz="0.0195 0 0.0215" rpy="0 0 1.5708" />
         <geometry>
           <box size="0.01 0.039 0.005" />
@@ -264,5 +264,5 @@
       </collision>
       <visual>
-        <origin xyz="-0.015 1.38778e-17 -0.007" rpy="3.914e-17 -8.32667e-17 1.5708" />
+        <origin xyz="-0.015 0 -0.007" rpy="0 0 1.5708" />
         <geometry>
           <mesh filename="package://gripper_description/mesh/rod_inner_bottom.stl" />
@@ -273,5 +273,5 @@
       </visual>
       <collision>
-        <origin xyz="0.02 2.08167e-18 -0.022" rpy="3.914e-17 -8.32667e-17 1.5708" />
+        <origin xyz="0.02 0 -0.022" rpy="0 0 1.5708" />
         <geometry>
           <box size="0.012 0.036 0.005" />
@@ -279,5 +279,5 @@
       </collision>
       <collision>
-        <origin xyz="0 7.63278e-18 -0.022" rpy="-3.914e-17 -8.32667e-17 1.5708" />
+        <origin xyz="0 0 -0.022" rpy="0 0 1.5708" />
         <geometry>
           <cylinder length="0.005" radius="0.011" />
@@ -292,5 +292,5 @@
     <link name="${ns}/rhs_claw">
       <visual>
-        <origin xyz="-6.93889e-18 -0.006 -4.93038e-32" rpy="0 -0 1.42883e-30" />
+        <origin xyz="0 -0.006 0" rpy="0 0 0" />
         <geometry>
           <mesh filename="package://gripper_description/mesh/jaw_plate.stl" />
@@ -301,5 +301,5 @@
       </visual>
       <collision>
-        <origin xyz="-6.93889e-18 -0.006 -4.93038e-32" rpy="0 -0 1.42883e-30" />
+        <origin xyz="0 -0.006 0" rpy="0 0 0" />
         <geometry>
           <mesh filename="package://gripper_description/mesh/jaw_plate.stl" />
@@ -312,9 +312,9 @@
         <origin xyz="0.00954335 0.0109092 -3.55182e-09" rpy="0 0 0" />
         <mass value="0.0706194" />
-        <inertia ixx="1.06828e-05" ixy="6.2682e-06" ixz="7.52244e-13" iyy="3.9212e-05" iyz="1.29448e-11" izz="3.75191e-05" />
+        <inertia ixx="1.06828e-05" ixy="6.2682e-06" ixz="0" iyy="3.9212e-05" iyz="1.29448e-11" izz="3.75191e-05" />
       </inertial>
     </link>
     <joint name="${ns}/rhs_j3" type="continuous">
-      <origin xyz="0.035 6.93889e-18 -3.46945e-18" rpy="-3.14159 -0 1.5708" />
+      <origin xyz="0.035 0 0" rpy="-3.14159 0 1.5708" />
       <parent link="${ns}/rhs_inner_beam" />
       <child link="${ns}/rhs_claw" />
@@ -325,5 +325,5 @@
     </joint>
     <joint name="${ns}/rhs_j1" type="continuous">
-      <origin xyz="0.03725 -0.015 8.67246e-31" rpy="-6.24854e-15 1.67434e-16 -1.5708" />
+      <origin xyz="0.03725 -0.015 0" rpy="0 0 -1.5708" />
       <parent link="${ns}/base_link" />
       <child link="${ns}/rhs_inner_beam" />
@@ -335,5 +335,5 @@
     <link name="${ns}/rhs_outer_beam">
       <visual>
-        <origin xyz="0.02 0.06 0.0025" rpy="3.14159 -0 1.42883e-30" />
+        <origin xyz="0.02 0.06 0.0025" rpy="3.14159 0 0" />
         <geometry>
           <mesh filename="package://gripper_description/mesh/rod_outer.stl" />
@@ -344,5 +344,5 @@
       </visual>
       <collision>
-        <origin xyz="1.04083e-17 0.0175 4.33681e-19" rpy="3.14159 -0 1.42883e-30" />
+        <origin xyz="0 0.0175 0" rpy="3.14159 0 0" />
         <geometry>
           <box size="0.01 0.043 0.005" />
@@ -350,11 +350,11 @@
       </collision>
       <inertial>
-        <origin xyz="1.04083e-17 0.0175 4.33681e-19" rpy="0 0 0" />
+        <origin xyz="0 0.0175 0" rpy="0 0 0" />
         <mass value="0.00168556" />
-        <inertia ixx="2.35764e-07" ixy="3.5459e-37" ixz="0" iyy="1.24039e-08" iyz="0" izz="2.41145e-07" />
+        <inertia ixx="2.35764e-07" ixy="0" ixz="0" iyy="1.24039e-08" iyz="0" izz="2.41145e-07" />
       </inertial>
     </link>
     <joint name="${ns}/rhs_j2" type="continuous">
-      <origin xyz="0.01725 -0.04 -3.46945e-18" rpy="-3.14159 6.24854e-15 -5.22162e-14" />
+      <origin xyz="0.01725 -0.04 0" rpy="-3.14159 0 0" />
       <parent link="${ns}/base_link" />
       <child link="${ns}/rhs_outer_beam" />

Commit message: added a TCP dummy link

File: gripper_description/urdf/gripper.reusable.xacro (robot description, xacro)
@@ -364,4 +364,10 @@
       <mimic joint="${ns}/lhs_j1" multiplier="1" offset="0" />
     </joint>
+    <joint name="${ns}/Base2TCP" type="fixed">
+      <origin xyz="0.098 0 0" rpy="0 0 0" />
+      <parent link="${ns}/base_link" />
+      <child link="${ns}/TCP" />
+    </joint>
+    <link name="${ns}/TCP" />
     <transmission name="${ns}/lhs_j1_transmission">
       <type>transmission_interface/SimpleTransmission</type>

File: gripper_description/urdf/gripper_0dof.reusable.xacro (robot description, xacro)
@@ -263,4 +263,10 @@
       </collision>
     </link>
+    <joint name="${ns}/Base2TCP" type="fixed">
+      <origin xyz="0.098 0 0" rpy="0 0 0" />
+      <parent link="${ns}/base_link" />
+      <child link="${ns}/TCP" />
+    </joint>
+    <link name="${ns}/TCP" />
   </xacro:macro>
 </robot>
